File: RobotTraceStopwatch/コード・配線/RobotTraceStopWatch.sch (EAGLE design)
At the start: 18 parts, among them U1 ESP-WROOM-32

Commit message: no message
Parts:
- added C1: 0.1u, 0my_lbr:C
- added C2: DNP, 0my_lbr:C
- added C3: 0.01u, 0my_lbr:C
- added R11, R12: 10k, 0my_lbr:R-US_0204/7
- added S1, S2: (no value), 0my_lbr:10-XX
Connections:
- new net N$21: R12.2, S2.S, S2.S1, U1.IO0
- new net N$24: C3.1, R11.2, S1.S, S1.S1, U1.EN(RST)
- net +3V3: now also C1.1, C2.1, R11.1, R12.1, U1.3V3
- net GND: now also C1.2, C2.2, C3.2, S1.P, S1.P1, S2.P, S2.P1, U1.GND@1, U1.GND@15, U1.GND@38
Other:
- moved on the sheet: FIRST_D1, FIRST_D2, LAST_D1, LAST_D2, R1, R2, R3, R4, R7, R8, R9
